File: ISA_DualUART.kicad_pcb (KiCad board)
At the start: 2 copper layers, 35 parts, among them J1 ISA BUS, J2 ADDR_IRQ, J3 UART1_SEL, J4 UART2_SEL, J5 Serial 1 IDC, J6 Serial 2 IDC, J7 Serial 1 DB9, U1 74LS138, U2 74LS138, U3 16550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

Commit message: First version of schematic for multifunction isa board
Parts:
- added C14: 51p, Capacitor_THT:C_Disc_D5.0mm_W2.5mm_P2.50mm, F.Cu at (48.6, 69.9)
- added C15: 51p, Capacitor_THT:C_Disc_D5.0mm_W2.5mm_P2.50mm, F.Cu at (40.4, 73.9)
- added C16: 51p, Capacitor_THT:C_Disc_D5.0mm_W2.5mm_P2.50mm, F.Cu at (56.7, 64.2)
- added C17: 51p, Capacitor_THT:C_Disc_D5.0mm_W2.5mm_P2.50mm, F.Cu at (56.7, 60.2)
- added C18: 10nF, Capacitor_THT:C_Disc_D5.0mm_W2.5mm_P2.50mm, F.Cu at (37.2, 82.0)
- added C19: 10nF, Capacitor_THT:C_Disc_D5.0mm_W2.5mm_P2.50mm, F.Cu at (37.2, 78.0)
- added C20: 10nF, Capacitor_THT:C_Disc_D5.0mm_W2.5mm_P2.50mm, F.Cu at (29.0, 89.4)
- added C21: 10nF, Capacitor_THT:C_Disc_D5.0mm_W2.5mm_P2.50mm, F.Cu at (19.8, 96.6)
- added C22: 10nF, Capacitor_THT:C_Disc_D5.0mm_W2.5mm_P2.50mm, F.Cu at (29.0, 85.3)
- added C23: 100nF, Capacitor_THT:C_Disc_D6.0mm_W2.5mm_P5.00mm, F.Cu at (48.1, 65.8)
- added C24: 100nF, Capacitor_THT:C_Disc_D6.0mm_W2.5mm_P5.00mm, F.Cu at (48.1, 61.8)
- added C25: 100nF, Capacitor_THT:C_Disc_D6.0mm_W2.5mm_P5.00mm, F.Cu at (40.0, 69.9)
- added C26: 100nF, Capacitor_THT:C_Disc_D6.0mm_W2.5mm_P5.00mm, F.Cu at (17.0, 66.5)
- added C27: 2.2nF, Capacitor_THT:C_Disc_D5.0mm_W2.5mm_P5.00mm, F.Cu at (3.00, 92.4)
- added C28: 2.2nF, Capacitor_THT:C_Disc_D5.0mm_W2.5mm_P5.00mm, F.Cu at (54.9, 56.1)
- added C29: 2.2nF, Capacitor_THT:C_Disc_D5.0mm_W2.5mm_P5.00mm, F.Cu at (28.6, 77.2)
- added C30: 2.2nF, Capacitor_THT:C_Disc_D5.0mm_W2.5mm_P5.00mm, F.Cu at (40.0, 65.8)
- added C31: 2.2nF, Capacitor_THT:C_Disc_D5.0mm_W2.5mm_P5.00mm, F.Cu at (40.0, 61.8)
- added C32: 2.2nF, Capacitor_THT:C_Disc_D5.0mm_W2.5mm_P5.00mm, F.Cu at (11.2, 96.6)
- added C33: 2.2nF, Capacitor_THT:C_Disc_D5.0mm_W2.5mm_P5.00mm, F.Cu at (54.9, 52.1)
- added C34: 2.2nF, Capacitor_THT:C_Disc_D5.0mm_W2.5mm_P5.00mm, F.Cu at (53.2, 48.0)
- added C35: 2.2nF, Capacitor_THT:C_Disc_D5.0mm_W2.5mm_P5.00mm, F.Cu at (3.00, 96.6)
- added J10: Parallel Port, Connector_PinSocket_2.54mm:PinSocket_2x13_P2.54mm_Vertical, F.Cu at (-45.2, 38.6)
- added J8: Game Port, Connector_PinHeader_2.54mm:PinHeader_2x08_P2.54mm_Vertical, F.Cu at (-36.2, 65.6)
- added JP1: Address selection, Connector_PinHeader_2.54mm:PinHeader_1x02_P2.54mm_Vertical, F.Cu at (58.6, 38.6)
- added JP2: Parport type, Connector_PinHeader_2.54mm:PinHeader_1x03_P2.54mm_Vertical, F.Cu at (53.9, 38.6)
- added R10: 4.7k, Resistor_THT:R_Axial_DIN0207_L6.3mm_D2.5mm_P10.16mm_Horizontal, F.Cu at (-23.6, 95.5)
- added R11: 4.7k, Resistor_THT:R_Axial_DIN0207_L6.3mm_D2.5mm_P10.16mm_Horizontal, F.Cu at (-10.3, 88.3)
- added R12: 4.7k, Resistor_THT:R_Axial_DIN0207_L6.3mm_D2.5mm_P10.16mm_Horizontal, F.Cu at (-10.3, 96.4)
- added R13: 4.7k, Resistor_THT:R_Axial_DIN0207_L6.3mm_D2.5mm_P10.16mm_Horizontal, F.Cu at (3.00, 88.3)
- added R14: 4.7k, Resistor_THT:R_Axial_DIN0207_L6.3mm_D2.5mm_P10.16mm_Horizontal, F.Cu at (41.6, 57.7)
- added R15: 4.7k, Resistor_THT:R_Axial_DIN0207_L6.3mm_D2.5mm_P10.16mm_Horizontal, F.Cu at (-36.9, 87.7)
- added R5: 2.2k, Resistor_THT:R_Axial_DIN0207_L6.3mm_D2.5mm_P10.16mm_Horizontal, F.Cu at (-10.3, 92.4)
- added R6: 2.2k, Resistor_THT:R_Axial_DIN0207_L6.3mm_D2.5mm_P10.16mm_Horizontal, F.Cu at (-36.9, 91.8)
- added R7: 2.2k, Resistor_THT:R_Axial_DIN0207_L6.3mm_D2.5mm_P10.16mm_Horizontal, F.Cu at (-36.9, 95.8)
- added R8: 2.2k, Resistor_THT:R_Axial_DIN0207_L6.3mm_D2.5mm_P10.16mm_Horizontal, F.Cu at (-23.6, 87.4)
- added R9: 4.7k, Resistor_THT:R_Axial_DIN0207_L6.3mm_D2.5mm_P10.16mm_Horizontal, F.Cu at (-23.6, 91.4)
- added RN1: 10k, Resistor_THT:R_Array_SIP9, F.Cu at (5.67, 42.8)
- added RN2: 4.7k, Resistor_THT:R_Array_SIP9, F.Cu at (5.67, 38.5)
- added U10: 74LS32, Package_DIP:DIP-14_W7.62mm_LongPads, F.Cu at (28.8, 57.9)
- added U11: 74LS30, Package_DIP:DIP-14_W7.62mm_LongPads, F.Cu at (5.78, 69.0)
- added U12: 74LS86, Package_DIP:DIP-14_W7.62mm_LongPads, F.Cu at (42.0, 38.4)
- added U13: 74LS02, Package_DIP:DIP-14_W7.62mm_LongPads, F.Cu at (17.4, 77.3)
- added U14: 74LS155, Package_DIP:DIP-16_W7.62mm_LongPads, F.Cu at (5.42, 47.1)
- added U15: 74LS245, Package_DIP:DIP-20_W7.62mm_LongPads, F.Cu at (-29.4, 38.4)
- added U16: 74LS174, Package_DIP:DIP-16_W7.62mm_Socket_LongPads, F.Cu at (-17.5, 65.4)
- added U18: 74LS05, Package_DIP:DIP-14_W7.62mm_Socket_LongPads, F.Cu at (17.1, 47.1)
- added U19: 74LS125, Package_DIP:DIP-14_W7.62mm_Socket_LongPads, F.Cu at (30.3, 38.4)
- added U20: 74LS240, Package_DIP:DIP-20_W7.62mm_LongPads, F.Cu at (-41.0, 38.4)
- added U21: 74LS244, Package_DIP:DIP-20_W7.62mm_LongPads, F.Cu at (-48.1, 73.5)
- added U3: 74LS32, Package_DIP:DIP-14_W7.62mm_LongPads, F.Cu at (-5.83, 69.0)
- added U7: NE558, Package_DIP:DIP-16_W7.62mm_Socket_LongPads, F.Cu at (-29.2, 65.4)
- added U8: 74LS688, Package_DIP:DIP-20_W7.62mm_LongPads, F.Cu at (-6.17, 38.4)
- added U9: 74HC244, Package_DIP:DIP-20_W7.62mm_LongPads, F.Cu at (-17.8, 38.4)
- moved C13 164.0 mm to (17.0, 70.6)
- moved C12 141.6 mm to (28.6, 81.3)
- renumbered U3 to U22

Commit message: Fix RPB line
Parts:
- added C36: 100nF, Capacitor_THT:C_Disc_D6.0mm_W2.5mm_P5.00mm, F.Cu at (-15.2, 11.4)
- added C37: 100nF, Capacitor_THT:C_Disc_D6.0mm_W2.5mm_P5.00mm, F.Cu at (-15.2, 15.5)
- added C38: 100nF, Capacitor_THT:C_Disc_D6.0mm_W2.5mm_P5.00mm, F.Cu at (-7.09, 11.4)
- added C39: 100nF, Capacitor_THT:C_Disc_D6.0mm_W2.5mm_P5.00mm, F.Cu at (-15.2, 19.5)
- added C40: 100nF, Capacitor_THT:C_Disc_D6.0mm_W2.5mm_P5.00mm, F.Cu at (-7.09, 15.5)
- added C41: 100nF, Capacitor_THT:C_Disc_D6.0mm_W2.5mm_P5.00mm, F.Cu at (-15.2, 23.6)
- added C42: 100nF, Capacitor_THT:C_Disc_D6.0mm_W2.5mm_P5.00mm, F.Cu at (1.06, 11.4)
- added C43: 100nF, Capacitor_THT:C_Disc_D6.0mm_W2.5mm_P5.00mm, F.Cu at (-7.09, 19.5)
- added C44: 100nF, Capacitor_THT:C_Disc_D6.0mm_W2.5mm_P5.00mm, F.Cu at (1.06, 15.5)
- added C45: 100nF, Capacitor_THT:C_Disc_D6.0mm_W2.5mm_P5.00mm, F.Cu at (-7.09, 23.6)
- added C46: 100nF, Capacitor_THT:C_Disc_D6.0mm_W2.5mm_P5.00mm, F.Cu at (1.06, 19.5)
- added C47: 100nF, Capacitor_THT:C_Disc_D6.0mm_W2.5mm_P5.00mm, F.Cu at (1.06, 23.6)
- J5, J6: footprint Connector_PinHeader_2.54mm:PinHeader_2x04_P2.54mm_Vertical -> Connector_PinHeader_2.54mm:PinHeader_2x05_P2.54mm_Vertical
Connections:
- U6 pad 9: (no net) -> /RS232_2_RI

Commit message: Begin organizing the board
Parts:
- removed J5: Serial 1 IDC, Connector_PinHeader_2.54mm:PinHeader_2x05_P2.54mm_Vertical
- added J9: Parport IRQ Select, Connector_PinHeader_2.54mm:PinHeader_2x04_P2.54mm_Vertical, F.Cu at (55.2, -3.17)
- added SW1: GP Address, Package_DIP:DIP-16_W7.62mm_LongPads, F.Cu at (43.3, -3.42)
- added U17: 74LS374, Package_DIP:DIP-20_W7.62mm_LongPads, F.Cu at (-55.9, 108.0)
- moved J7 199.5 mm to (304.8, 167.0), turned to 90 degrees
- moved U4 178.1 mm to (245.1, 174.6), turned to 90 degrees
- moved U5 172.0 mm to (288.9, 125.7), turned to 270 degrees
- moved C8 148.7 mm to (271.1, 182.2), turned to 270 degrees
- moved J6 145.2 mm to (305.4, 111.8), turned to 90 degrees
- moved U2 144.8 mm to (275.6, 188.6), turned to 90 degrees
- moved U1 142.3 mm to (245.7, 188.6), turned to 90 degrees
- moved C9 122.6 mm to (240.0, 169.5), turned to 90 degrees
- moved C11 122.1 mm to (240.0, 143.5), turned to 270 degrees
- moved U6 117.8 mm to (257.2, 125.7), turned to 270 degrees
- moved C7 115.6 mm to (241.3, 182.2), turned to 270 degrees
- moved U22 112.7 mm to (245.1, 153.7), turned to 90 degrees
- moved X1 82.9 mm to (218.4, 148.6)
Connections:
- JP2 pad 2: (no net) -> Net-(JP2-Pad2)
- U14 pad 9: (no net) -> /PARPORT_WPA
- U19 pad 10: /PARPORT_RPB -> /PARPORT_RPC
- U19 pad 11: (no net) -> Net-(J9-Pad2)

Commit message: First model of the board
Parts:
- removed C17: 51p, Capacitor_THT:C_Disc_D5.0mm_W2.5mm_P2.50mm
- removed C18, C19, C20, C21, C22: 10nF, Capacitor_THT:C_Disc_D5.0mm_W2.5mm_P2.50mm
- removed C23, C24, C25, C26, C42, C43, C44, C45, C46, C47: 100nF, Capacitor_THT:C_Disc_D6.0mm_W2.5mm_P5.00mm
- removed J8: Game Port, Connector_PinHeader_2.54mm:PinHeader_2x08_P2.54mm_Vertical
- removed R5, R6, R7, R8: 2.2k, Resistor_THT:R_Axial_DIN0207_L6.3mm_D2.5mm_P10.16mm_Horizontal
- removed RN1: 10k, Resistor_THT:R_Array_SIP9
- removed RN2: 4.7k, Resistor_THT:R_Array_SIP9
- removed SW1: GP Address, Package_DIP:DIP-16_W7.62mm_LongPads
- removed U10, U3: 74LS32, Package_DIP:DIP-14_W7.62mm_LongPads
- removed U7: NE558, Package_DIP:DIP-16_W7.62mm_Socket_LongPads
- removed U8: 74LS688, Package_DIP:DIP-20_W7.62mm_LongPads
- removed U9: 74HC244, Package_DIP:DIP-20_W7.62mm_LongPads
- C14, C15, C16: value 51p -> 100nF; footprint Capacitor_THT:C_Disc_D5.0mm_W2.5mm_P2.50mm -> Capacitor_THT:C_Disc_D6.0mm_W2.5mm_P5.00mm
- J7: footprint Connector_Dsub:DSUB-9_Male_Horizontal_P2.77x2.84mm_EdgePinOffset4.94mm_Housed_MountingHolesOffset7.48mm -> Connector_Dsub:DSUB-9_Male_Horizontal_P2.77x2.84mm_EdgePinOffset7.70mm_Housed_MountingHolesOffset9.12mm
- moved U20 287.6 mm to (215.9, 167.6), turned to 270 degrees
- moved U15 284.0 mm to (215.9, 181.6), turned to 270 degrees
- moved C41 280.0 mm to (221.0, 174.0), turned to 90 degrees
- moved U17 275.6 mm to (215.9, 153.7), turned to 270 degrees
- moved U21 272.2 mm to (215.9, 139.7), turned to 270 degrees
- moved C40 260.4 mm to (188.0, 188.0), turned to 90 degrees
- moved J9 257.3 mm to (226.1, 189.2), turned to 90 degrees
- moved C39 256.3 mm to (189.2, 174.0), turned to 90 degrees
- moved J10 252.8 mm to (194.3, 119.4), turned to 270 degrees
- moved C38 241.2 mm to (162.6, 182.9), turned to 270 degrees
- moved C36 240.9 mm to (162.6, 174.0), turned to 90 degrees
- moved C37 229.1 mm to (162.6, 160.0), turned to 90 degrees
- moved C35 221.3 mm to (221.0, 134.6), turned to 90 degrees
- moved C12 217.6 mm to (221.0, 182.9), turned to 270 degrees
- moved U14 216.6 mm to (185.4, 167.6), turned to 270 degrees
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Connections:
- C12 pad 1: VCC -> GND
- C12 pad 2: GND -> VCC
- C14 pad 1: /J1B1 -> VCC
- C15 pad 1: /J1B2 -> VCC
- C16 pad 1: /J2B1 -> VCC
- U12 pad 10: /PARPORT_IRQEN -> VCC
- U12 pad 9: VCC -> /PARPORT_IRQEN
Other:
- board outline added: 176.5 x 90.2 mm
- net class POWER added: clearance 0.2, trace_width 0.4, via_dia 0.8, via_drill 0.4
- net class POWR_SMALL added: clearance 0.2, trace_width 0.3, via_dia 0.8, via_drill 0.4
