File: ISA_DualUART.sch (KiCad schematic (older format))
At the start: 86 parts, among them J1 ISA BUS, J2 ADDR_IRQ, J3 UART1_SEL, J4 UART2_SEL, J5 Serial 1 IDC, J6 Serial 2 IDC, J7 Serial 1 DB9, J8 Game Port, SW1 GP Address, U1 74LS138, U10 74LS32, U11 74LS30, U12 74LS86, U13 74LS02, U14 74LS155, U15 74LS245, U16 74LS174, U17 74LS374, U18 74LS05, U2 74LS138, U3 74LS32, U4 16550, U5 GD75232N, U6 GD75232N, U7 NE558, U8 74LS688, U9 74HC244, X1 1.8432Mhz

Commit message: First version of schematic for multifunction isa board
Parts:
- added C36, C37, C38, C39, C40, C41, C42, C43, C44, C45, C46, C47: 100nF, Capacitor_THT:C_Disc_D6.0mm_W2.5mm_P5.00mm, symbol Device:C_Small
- added J10: Parallel Port, Connector_PinSocket_2.54mm:PinSocket_2x13_P2.54mm_Vertical, symbol Connector_Generic:Conn_02x13_Odd_Even
- added J9: Parport IRQ Select, symbol Connector_Generic:Conn_02x04_Odd_Even
- added unit 4 of U12
- added unit 1 of U12
- added unit 1 of U13
- added unit 6 of U18
- added U19: 74LS125, Package_DIP:DIP-14_W7.62mm_Socket_LongPads, symbol 74xx:74LS125
- added U20: 74LS240, Package_DIP:DIP-20_W7.62mm_LongPads, symbol 74xx:74LS240
- added U21: 74LS244, Package_DIP:DIP-20_W7.62mm_LongPads, symbol 74xx:74LS244
- J5, J6: footprint Connector_PinHeader_2.54mm:PinHeader_2x04_P2.54mm_Vertical -> Connector_PinHeader_2.54mm:PinHeader_2x05_P2.54mm_Vertical
- U22: renamed from U3; value 74LS32 -> 16550; footprint Package_DIP:DIP-14_W7.62mm_LongPads -> Package_DIP:DIP-40_W15.24mm_LongPads
Connections:
- net GND: now also C36.2, C37.2, C38.2, C39.2, C40.2, C41.2, C42.2, C43.2, C44.2, C45.2, C46.2, C47.2, J10.18 (Pin_18), J10.19 (Pin_19), J10.20 (Pin_20), J10.21 (Pin_21), J10.22 (Pin_22), J10.23 (Pin_23), J10.24 (Pin_24), J10.25 (Pin_25), U19.7 (GND), U20.10 (GND), U21.10 (GND)
- net IRQ3: now also J9.1 (Pin_1)
- net IRQ4: now also J9.3 (Pin_3)
- net IRQ5: now also J9.5 (Pin_5)
- net IRQ7: now also J9.7 (Pin_7)
- net PARPORT_BD0: now also U20.3 (O3b), U21.3 (O3b)
- net PARPORT_BD1: now also U20.5 (O2b), U21.5 (O2b)
- net PARPORT_BD2: now also U20.7 (O1b), U21.7 (O1b)
- net PARPORT_BD3: now also U19.6, U20.9 (O0b), U21.9 (O0b)
- net PARPORT_BD4: now also U19.8, U20.18 (O0a), U21.18 (O0a)
- net PARPORT_BD5: now also U20.16 (O1a), U21.16 (O1a)
- net PARPORT_BD6: now also U20.14 (O2a), U21.14 (O2a)
- net PARPORT_BD7: now also U20.12 (O3a), U21.12 (O3a)
- net PARPORT_DATA0: now also J10.2 (Pin_2), U21.17 (I3b)
- net PARPORT_DATA1: now also J10.3 (Pin_3), U21.15 (I2b)
- net PARPORT_DATA2: now also J10.4 (Pin_4), U21.13 (I1b)
- net PARPORT_DATA3: now also J10.5 (Pin_5), U21.11 (I0b)
- net PARPORT_DATA4: now also J10.6 (Pin_6), U21.2 (I0a)
- net PARPORT_DATA5: now also J10.7 (Pin_7), U21.4 (I1a)
- net PARPORT_DATA6: now also J10.8 (Pin_8), U21.6 (I2a)
- net PARPORT_DATA7: now also J10.9 (Pin_9), U21.8 (I3a)
- net PARPORT_IRQEN: now also U19.9
- net PARPORT_RPA: now also U21.1 (OEa), U21.19 (OEb)
- net PARPORT_RPB: now also U19.10, U19.4, U20.1 (OEa)
- net PARPORT_RPC: now also U20.19 (OEb)
- net VCC: now also U12.9, C36.1, C37.1, C38.1, C39.1, C40.1, C41.1, C42.1, C43.1, C44.1, C45.1, C46.1, C47.1, U12.12, U12.2, U19.1, U19.14 (VCC), U19.2, U20.20 (VCC), U21.20 (VCC)
- net ~PARPORT_AUTOFD: now also J10.14 (Pin_14), U20.15 (I2b)
- net ~PARPORT_INIT: now also J10.16 (Pin_16), U18.13
- net ~PARPORT_IRQEN: now also U19.13
- net ~PARPORT_SLCTIN: now also J10.17 (Pin_17), U20.11 (I0b)
- net ~PARPORT_STROBE: now also J10.1 (Pin_1), U20.17 (I3b)
- net at R15.2: now also U18.12, U20.13 (I1b); no longer U12.9
- new net: J9.2 (Pin_2), J9.4 (Pin_4), J9.6 (Pin_6), J9.8 (Pin_8), U19.11
- new net: U13.1, U20.2 (I0a)
- new net: U12.3, U20.4 (I1a)
- new net PARPORT_BUSY: J10.11 (Pin_11), U20.8 (I3a)
- new net PARPORT_IRQ: U12.11, U19.12, U20.6 (I2a)
- new net PARPORT_PE: J10.12 (Pin_12), U12.1
- new net PARPORT_SLCT: J10.13 (Pin_13), U13.2, U13.3
- new net ~PARPORT_ACK: J10.10 (Pin_10), U12.13
- new net ~PARPORT_ERROR: J10.15 (Pin_15), U19.5
- no-connect marks 45 -> 47
Other:
- moved on the sheet: C1, C10, C11, C12, C13, C2, C23, C24, C25, C26, C27, C28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

Commit message: Fix RPB line
Connections:
- net PARPORT_RPB: no longer U19.10
- net PARPORT_RPC: now also U19.10
Changed lines of the file:
@@
 $EndComp
 Text Label 18350 17050 0    50   ~ 0
-PARPORT_RPB
+PARPORT_RPC
 Wire Wire Line
 	18350 17050 19100 17050

Commit message: Begin organizing the board
Parts:
- removed J5: Serial 1 IDC, Connector_PinHeader_2.54mm:PinHeader_2x05_P2.54mm_Vertical, symbol Connector_Generic:Conn_02x05_Odd_Even
- J9: footprint (none) -> Connector_PinHeader_2.54mm:PinHeader_2x04_P2.54mm_Vertical
- SW1: footprint (none) -> Package_DIP:DIP-16_W7.62mm_LongPads
- U17: footprint (none) -> Package_DIP:DIP-20_W7.62mm_LongPads
Connections:
- no-connect marks 47 -> 46
Changed lines of the file:
@@
 	21200 2150 20700 2150
 Wire Wire Line
-	21300 2750 21300 2850
-Text Label 21200 2550 2    50   ~ 0
-RS232_1_RI
-Text Label 19700 2650 0    50   ~ 0
-RS232_1_CTS
-Text Label 21200 2650 2    50   ~ 0
-RS232_1_RTS
-Text Label 19700 2750 0    50   ~ 0
-RS232_1_DSR
-Wire Wire Line
-	20700 2750 21300 2750
-$Comp
-L power:GND #PWR0126
-U 1 1 605E18EB
-P 21300 2850
-F 0 "#PWR0126" H 21300 2600 50  0001 C CNN
-F 1 "GND" H 21305 2677 50  0000 C CNN
-F 2 "" H 21300 2850 50  0001 C CNN
-F 3 "" H 21300 2850 50  0001 C CNN
-	1    21300 2850
-	1    0    0    -1
-$EndComp
-Text Label 19700 2850 0    50   ~ 0
-RS232_1_DTR
-Text Label 21200 2850 2    50   ~ 0
-RS232_1_TX
-Text Label 19700 2950 0    50   ~ 0
-RS232_1_RX
-Text Label 21200 2950 2    50   ~ 0
-RS232_1_DCD
-NoConn ~ 20200 2550
-$Comp
-L Connector_Generic:Conn_02x05_Odd_Even J5
-U 1 1 605E18FA
-P 20500 2750
-F 0 "J5" H 20550 2325 50  0000 C CNN
-F 1 "Serial 1 IDC" H 20550 2416 50  0000 C CNN
-F 2 "Connector_PinHeader_2.54mm:PinHeader_2x05_P2.54mm_Vertical" H 20500 2750 50  0001 C CNN
-F 3 "~" H 20500 2750 50  0001 C CNN
-	1    20500 2750
-	-1   0    0    1
-$EndComp
-Wire Wire Line
-	20200 2650 19700 2650
-Wire Wire Line
-	20200 2750 19700 2750
-Wire Wire Line
-	20200 2850 19700 2850
-Wire Wire Line
-	20200 2950 19700 2950
-Wire Wire Line
-	21200 2550 20700 2550
-Wire Wire Line
-	21200 2650 20700 2650
-Wire Wire Line
-	21200 2850 20700 2850
-Wire Wire Line
-	21200 2950 20700 2950
-Wire Wire Line
 	2300 6550 1600 6550
 Wire Wire Line
@@
 F 0 "SW1" H 5700 8187 60  0000 C CNN
 F 1 "GP Address" H 5700 8081 60  0000 C CNN
-F 2 "" H 5700 7600 60  0000 C CNN
+F 2 "Package_DIP:DIP-16_W7.62mm_LongPads" H 5700 7600 60  0000 C CNN
 F 3 "" H 5700 7600 60  0000 C CNN
 	1    5700 7550
@@
 F 0 "U17" H 16350 10350 50  0000 C CNN
 F 1 "74LS374" H 16800 10350 50  0000 C CNN
-F 2 "" H 16600 9700 50  0001 C CNN
+F 2 "Package_DIP:DIP-20_W7.62mm_LongPads" H 16600 9700 50  0001 C CNN
 F 3 "http://www.ti.com/lit/gpn/sn74LS374" H 16600 9700 50  0001 C CNN
 	1    16600 9700
@@
 F 0 "J9" H 16050 15717 50  0000 C CNN
 F 1 "Parport IRQ Select" H 16050 15626 50  0000 C CNN
-F 2 "" H 16000 15400 50  0001 C CNN
+F 2 "Connector_PinHeader_2.54mm:PinHeader_2x04_P2.54mm_Vertical" H 16000 15400 50  0001 C CNN
 F 3 "~" H 16000 15400 50  0001 C CNN
 	1    16000 15400
@@
 $EndComp
 $Comp
-L power:GND #PWR?
+L power:GND #PWR0206
 U 1 1 737061C8
 P 1050 12300
-F 0 "#PWR?" H 1050 12050 50  0001 C CNN
+F 0 "#PWR0206" H 1050 12050 50  0001 C CNN
 F 1 "GND" H 1055 12127 50  0000 C CNN
 F 2 "" H 1050 12300 50  0001 C CNN
@@
 	1800 12300 1700 12300
 $Comp
-L power:VCC #PWR?
+L power:VCC #PWR0207
 U 1 1 737061D4
 P 1800 12300
-F 0 "#PWR?" H 1800 12150 50  0001 C CNN
+F 0 "#PWR0207" H 1800 12150 50  0001 C CNN
 F 1 "VCC" H 1815 12473 50  0000 C CNN
 F 2 "" H 1800 12300 50  0001 C CNN
@@
 $EndComp
 $Comp
-L power:GND #PWR?
+L power:GND #PWR0208
 U 1 1 73AD0116
 P 3600 12300
-F 0 "#PWR?" H 3600 12050 50  0001 C CNN
+F 0 "#PWR0208" H 3600 12050 50  0001 C CNN
 F 1 "GND" H 3605 12127 50  0000 C CNN
 F 2 "" H 3600 12300 50  0001 C CNN
@@
 	4350 12300 4250 12300
 $Comp
-L power:VCC #PWR?
+L power:VCC #PWR0209
 U 1 1 73AD0122
 P 4350 12300
-F 0 "#PWR?" H 4350 12150 50  0001 C CNN
+F 0 "#PWR0209" H 4350 12150 50  0001 C CNN
 F 1 "VCC" H 4365 12473 50  0000 C CNN
 F 2 "" H 4350 12300 50  0001 C CNN
@@
 Wire Wire Line
 	3700 14350 3700 14800
+Wire Notes Line
+	12800 17550 22700 17550
+Wire Notes Line
+	22700 17550 22700 5350
+Wire Notes Line
+	22700 5350 12800 5350
+Wire Notes Line
+	12800 5350 12800 17550
 Wire Bus Line
 	21550 7800 21550 13500

Commit message: First model of the board
Parts:
- removed C17: 51p, Capacitor_THT:C_Disc_D5.0mm_W2.5mm_P2.50mm, symbol Device:C_Small
- removed C18, C19, C20, C21, C22: 10nF, Capacitor_THT:C_Disc_D5.0mm_W2.5mm_P2.50mm, symbol Device:C_Small
- removed C23, C24, C25, C26, C42, C43, C44, C45, C46, C47: 100nF, Capacitor_THT:C_Disc_D6.0mm_W2.5mm_P5.00mm, symbol Device:C_Small
- removed J8: Game Port, Connector_PinHeader_2.54mm:PinHeader_2x08_P2.54mm_Vertical, symbol Connector_Generic:Conn_02x08_Odd_Even
- removed R5, R6, R7, R8: 2.2k, Resistor_THT:R_Axial_DIN0207_L6.3mm_D2.5mm_P10.16mm_Horizontal, symbol Device:R_Small
- removed RN1: 10k, Resistor_THT:R_Array_SIP9, symbol Device:R_Network08
- removed RN2: 4.7k, Resistor_THT:R_Array_SIP9, symbol Device:R_Network08
- removed SW1: GP Address, Package_DIP:DIP-16_W7.62mm_LongPads, symbol skiselev_libraries:Switch_DIP_8_Positions
- removed U10, U3: 74LS32, Package_DIP:DIP-14_W7.62mm_LongPads, symbol 74xx:74LS32
- removed U7: NE558, Package_DIP:DIP-16_W7.62mm_Socket_LongPads, symbol skiselev_libraries:NE558
- removed U8: 74LS688, Package_DIP:DIP-20_W7.62mm_LongPads, symbol 74xx:74LS688
- removed U9: 74HC244, Package_DIP:DIP-20_W7.62mm_LongPads, symbol 74xx:74HC244
- C14, C15, C16: value 51p -> 100nF; footprint Capacitor_THT:C_Disc_D5.0mm_W2.5mm_P2.50mm -> Capacitor_THT:C_Disc_D6.0mm_W2.5mm_P5.00mm
- J7: footprint Connector_Dsub:DSUB-9_Male_Horizontal_P2.77x2.84mm_EdgePinOffset4.94mm_Housed_MountingHolesOffset7.48mm -> Connector_Dsub:DSUB-9_Male_Horizontal_P2.77x2.84mm_EdgePinOffset7.70mm_Housed_MountingHolesOffset9.12mm
Connections:
- net J1B1 is gone; now on net VCC: C14.1
- net J1B2 is gone; now on net VCC: C15.1
- net J2B1 is gone; now on net VCC: C16.1
- net GND: now also C12.1; no longer C12.2
- net PARPORT_IRQEN: now also U12.9; no longer U12.10
- net VCC: now also C12.2, U12.10; no longer C12.1, U12.9
- no-connect marks 46 -> 43
Other:
- note added: "Parallel Port"
- note removed: "Gameport"
- moved on the sheet: C12, C27, C28, C29, C30, C31, C32, C33, C34, C35, C36, C37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

Commit message: Chane connector
Parts:
- J10: footprint Connector_PinSocket_2.54mm:PinSocket_2x13_P2.54mm_Vertical -> Connector_PinHeader_2.54mm:PinHeader_2x13_P2.54mm_Vertical
Changed lines of the file:
@@
 F 0 "J10" H 13550 7217 50  0000 C CNN
 F 1 "Parallel Port" H 13550 7126 50  0000 C CNN
-F 2 "Connector_PinSocket_2.54mm:PinSocket_2x13_P2.54mm_Vertical" H 13500 6400 50  0001 C CNN
+F 2 "Connector_PinHeader_2.54mm:PinHeader_2x13_P2.54mm_Vertical" H 13500 6400 50  0001 C CNN
 F 3 "~" H 13500 6400 50  0001 C CNN
 	1    13500 6400

Commit message: Add text and generate gerbers
Changed lines of the file:
@@
 EELAYER 30 0
 EELAYER END
-$Descr A1 33110 23386
+$Descr A2 23386 16535
 encoding utf-8
 Sheet 1 1
-Title ""
+Title "Serial + Parallel Port ISA Adapterr"
 Date ""
 Rev "1.0"
@@
 Connection ~ 13800 13500
 Wire Notes Line
-	5050 15900 22700 15900
-Wire Notes Line
-	22700 15900 22700 5350
-Wire Notes Line
 	5050 5350 22700 5350
 Wire Notes Line
 	5050 5350 5050 15900
-Text Notes 20650 15800 0    197  ~ 0
+Text Notes 20550 14550 0    197  ~ 0
 Parallel Port
 Wire Wire Line
@@
 Wire Wire Line
 	1350 14400 1800 14400
+Wire Notes Line
+	5050 15900 18550 15900
+Wire Notes Line
+	18550 15900 18550 14700
+Wire Notes Line
+	18550 14700 22700 14700
+Wire Notes Line
+	22700 14700 22700 5350
 Wire Bus Line
 	13800 7800 13800 13500

Commit message: Change socket footprint to normal DIP
Parts:
- U16: footprint Package_DIP:DIP-16_W7.62mm_Socket_LongPads -> Package_DIP:DIP-16_W7.62mm_LongPads
- U18, U19: footprint Package_DIP:DIP-14_W7.62mm_Socket_LongPads -> Package_DIP:DIP-14_W7.62mm_LongPads
Changed lines of the file:
@@
 F 0 "U16" H 8600 12650 50  0000 C CNN
 F 1 "74LS174" H 9100 12650 50  0000 C CNN
-F 2 "Package_DIP:DIP-16_W7.62mm_Socket_LongPads" H 8850 12100 50  0001 C CNN
+F 2 "Package_DIP:DIP-16_W7.62mm_LongPads" H 8850 12100 50  0001 C CNN
 F 3 "http://www.ti.com/lit/gpn/sn74LS174" H 8850 12100 50  0001 C CNN
 	1    8850 12100
@@
 F 0 "U18" H 6630 13096 50  0000 L CNN
 F 1 "74LS05" H 6630 13005 50  0000 L CNN
-F 2 "Package_DIP:DIP-14_W7.62mm_Socket_LongPads" H 6400 13050 50  0001 C CNN
+F 2 "Package_DIP:DIP-14_W7.62mm_LongPads" H 6400 13050 50  0001 C CNN
 F 3 "http://www.ti.com/lit/gpn/sn74LS05" H 6400 13050 50  0001 C CNN
 	7    6400 13050
@@
 F 0 "U18" H 10000 11317 50  0000 C CNN
 F 1 "74LS05" H 10000 11226 50  0000 C CNN
-F 2 "Package_DIP:DIP-14_W7.62mm_Socket_LongPads" H 10000 11000 50  0001 C CNN
+F 2 "Package_DIP:DIP-14_W7.62mm_LongPads" H 10000 11000 50  0001 C CNN
 F 3 "http://www.ti.com/lit/gpn/sn74LS05" H 10000 11000 50  0001 C CNN
 	1    10000 11000
@@
 F 0 "U18" H 10000 11767 50  0000 C CNN
 F 1 "74LS05" H 10000 11676 50  0000 C CNN
-F 2 "Package_DIP:DIP-14_W7.62mm_Socket_LongPads" H 10000 11450 50  0001 C CNN
+F 2 "Package_DIP:DIP-14_W7.62mm_LongPads" H 10000 11450 50  0001 C CNN
 F 3 "http://www.ti.com/lit/gpn/sn74LS05" H 10000 11450 50  0001 C CNN
 	3    10000 11450
@@
 F 0 "U18" H 10650 12217 50  0000 C CNN
 F 1 "74LS05" H 10650 12126 50  0000 C CNN
-F 2 "Package_DIP:DIP-14_W7.62mm_Socket_LongPads" H 10650 11900 50  0001 C CNN
+F 2 "Package_DIP:DIP-14_W7.62mm_LongPads" H 10650 11900 50  0001 C CNN
 F 3 "http://www.ti.com/lit/gpn/sn74LS05" H 10650 11900 50  0001 C CNN
 	2    10650 11900
@@
 F 0 "U18" H 11750 12217 50  0000 C CNN
 F 1 "74LS05" H 11750 12126 50  0000 C CNN
-F 2 "Package_DIP:DIP-14_W7.62mm_Socket_LongPads" H 11750 11900 50  0001 C CNN
+F 2 "Package_DIP:DIP-14_W7.62mm_LongPads" H 11750 11900 50  0001 C CNN
 F 3 "http://www.ti.com/lit/gpn/sn74LS05" H 11750 11900 50  0001 C CNN
 	5    11750 11900
@@
 F 0 "U18" H 10650 12717 50  0000 C CNN
 F 1 "74LS05" H 10650 12626 50  0000 C CNN
-F 2 "Package_DIP:DIP-14_W7.62mm_Socket_LongPads" H 10650 12400 50  0001 C CNN
+F 2 "Package_DIP:DIP-14_W7.62mm_LongPads" H 10650 12400 50  0001 C CNN
 F 3 "http://www.ti.com/lit/gpn/sn74LS05" H 10650 12400 50  0001 C CNN
 	4    10650 12400
@@
 F 0 "U19" H 7380 13096 50  0000 L CNN
 F 1 "74LS125" H 7380 13005 50  0000 L CNN
-F 2 "Package_DIP:DIP-14_W7.62mm_Socket_LongPads" H 7150 13050 50  0001 C CNN
+F 2 "Package_DIP:DIP-14_W7.62mm_LongPads" H 7150 13050 50  0001 C CNN
 F 3 "http://www.ti.com/lit/gpn/sn74LS125" H 7150 13050 50  0001 C CNN
 	5    7150 13050
@@
 F 0 "U19" H 15300 9067 50  0000 C CNN
 F 1 "74LS125" H 15300 8976 50  0000 C CNN
-F 2 "Package_DIP:DIP-14_W7.62mm_Socket_LongPads" H 15300 8750 50  0001 C CNN
+F 2 "Package_DIP:DIP-14_W7.62mm_LongPads" H 15300 8750 50  0001 C CNN
 F 3 "http://www.ti.com/lit/gpn/sn74LS125" H 15300 8750 50  0001 C CNN
 	4    15300 8750
@@
 F 0 "U18" H 17100 9567 50  0000 C CNN
 F 1 "74LS05" H 17100 9476 50  0000 C CNN
-F 2 "Package_DIP:DIP-14_W7.62mm_Socket_LongPads" H 17100 9250 50  0001 C CNN
+F 2 "Package_DIP:DIP-14_W7.62mm_LongPads" H 17100 9250 50  0001 C CNN
 F 3 "http://www.ti.com/lit/gpn/sn74LS05" H 17100 9250 50  0001 C CNN
 	6    17100 9250
@@
 F 0 "U19" H 18100 10317 50  0000 C CNN
 F 1 "74LS125" H 18100 10226 50  0000 C CNN
-F 2 "Package_DIP:DIP-14_W7.62mm_Socket_LongPads" H 18100 10000 50  0001 C CNN
+F 2 "Package_DIP:DIP-14_W7.62mm_LongPads" H 18100 10000 50  0001 C CNN
 F 3 "http://www.ti.com/lit/gpn/sn74LS125" H 18100 10000 50  0001 C CNN
 	2    18100 10000
@@
 F 0 "U19" H 18100 11117 50  0000 C CNN
 F 1 "74LS125" H 18100 11026 50  0000 C CNN
-F 2 "Package_DIP:DIP-14_W7.62mm_Socket_LongPads" H 18100 10800 50  0001 C CNN
+F 2 "Package_DIP:DIP-14_W7.62mm_LongPads" H 18100 10800 50  0001 C CNN
 F 3 "http://www.ti.com/lit/gpn/sn74LS125" H 18100 10800 50  0001 C CNN
 	3    18100 10800
@@
 F 0 "U19" H 7600 15167 50  0000 C CNN
 F 1 "74LS125" H 7600 15076 50  0000 C CNN
-F 2 "Package_DIP:DIP-14_W7.62mm_Socket_LongPads" H 7600 14850 50  0001 C CNN
+F 2 "Package_DIP:DIP-14_W7.62mm_LongPads" H 7600 14850 50  0001 C CNN
 F 3 "http://www.ti.com/lit/gpn/sn74LS125" H 7600 14850 50  0001 C CNN
 	1    7600 14850
